File: rfid-control-acceso-eest3/06_cerradura_12v.kicad_sch (KiCad schematic)
At the start: 7 parts, among them J9 LOCK_12V_1.8A_21.6W, Q2 AO3400A_PRELIM

Commit message: Corrige tres diodos invertidos, netclasses y recalcula el floorplan
Errores electricos, verificados regenerando el netlist con kicad-cli:

- D1 tenia el catodo en +12V_IN y el anodo hacia F1, o sea bloqueaba la
  polaridad correcta. Montado asi la placa no encendia.
- D2 y D3 tenian el anodo a GND y el catodo hacia R3/R4. Como un GPIO nunca
  baja de 0 V, los LEDs no podian encender.
- La red entre D1 y F1 no coincidia con ningun patron de netclass y heredaba
  Default: 0,2 mm de pista para ~2,2 A. Pasa a LOCK_POWER (2,0 mm), igual que
  +12V_IN, que estaba en POWER_12V_AUX (0,8 mm).
- Al girar los LEDs, KiCad renombro las redes autogeneradas. Las netclasses
  apuntaban a los nombres viejos; se re-apuntaron.

Footprints: se eliminan los ocho PLACEHOLDER_NO_FABRICAR. Todos tenian
equivalente real ya instalado en KiCad 10. C9 pasa a MLCC 1206: tenia simbolo
no polarizado con footprint de electrolitico. El unico footprint local que
queda es el del ESP32-S3, con la hilera par duplicada en 22,86 y 25,40 mm
porque no se midio el modulo fisico. El paso doble cubre la separacion, no el
orden de pines: hay que verificar 3V3, EN, 5V y GND por continuidad antes de
soldar.

Floorplan: la posicion real de los pines de J13 determina el orden de los
bloques, y estaban casi invertidos. Lazo de potencia J1-J9 de 86 a 38 mm,
estrella de masa NT1-J1 de 60 a 9 mm, SPI de ~70 a 8,7 mm. Contorno de 120x80
a 140x100 mm: la densidad bajaba de 53% a 36% y la caja sigue sin definir.

Sigue sin ruteo, sin vias y sin archivos de fabricacion. Falta ejecutar
Update PCB from Schematic en la GUI: KiCad no expone esa operacion por CLI.

Co-Authored-By: Claude Opus 5 <noreply@anthropic.com>
Parts:
- J9: footprint rfid_eest3:KF301_2P_P5.08_PLACEHOLDER_NO_FABRICAR -> TerminalBlock_RND:TerminalBlock_RND_205-00232_1x02_P5.08mm_Horizontal
Changed lines of the file:
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@@
 			)
 		)
-		(property "Footprint" "rfid_eest3:KF301_2P_P5.08_PLACEHOLDER_NO_FABRICAR"
+		(property "Footprint" "TerminalBlock_RND:TerminalBlock_RND_205-00232_1x02_P5.08mm_Horizontal"
 			(at 180.34 54.61 0)
 			(hide yes)
