File: rfid-control-acceso-eest3/03_rfid_rc522.kicad_sch (KiCad schematic)
At the start: 12 parts, among them J5 RC522_8PIN_3V3_PINOUT_PENDING

Commit message: Corrige tres diodos invertidos, netclasses y recalcula el floorplan
Errores electricos, verificados regenerando el netlist con kicad-cli:

- D1 tenia el catodo en +12V_IN y el anodo hacia F1, o sea bloqueaba la
  polaridad correcta. Montado asi la placa no encendia.
- D2 y D3 tenian el anodo a GND y el catodo hacia R3/R4. Como un GPIO nunca
  baja de 0 V, los LEDs no podian encender.
- La red entre D1 y F1 no coincidia con ningun patron de netclass y heredaba
  Default: 0,2 mm de pista para ~2,2 A. Pasa a LOCK_POWER (2,0 mm), igual que
  +12V_IN, que estaba en POWER_12V_AUX (0,8 mm).
- Al girar los LEDs, KiCad renombro las redes autogeneradas. Las netclasses
  apuntaban a los nombres viejos; se re-apuntaron.

Footprints: se eliminan los ocho PLACEHOLDER_NO_FABRICAR. Todos tenian
equivalente real ya instalado en KiCad 10. C9 pasa a MLCC 1206: tenia simbolo
no polarizado con footprint de electrolitico. El unico footprint local que
queda es el del ESP32-S3, con la hilera par duplicada en 22,86 y 25,40 mm
porque no se midio el modulo fisico. El paso doble cubre la separacion, no el
orden de pines: hay que verificar 3V3, EN, 5V y GND por continuidad antes de
soldar.

Floorplan: la posicion real de los pines de J13 determina el orden de los
bloques, y estaban casi invertidos. Lazo de potencia J1-J9 de 86 a 38 mm,
estrella de masa NT1-J1 de 60 a 9 mm, SPI de ~70 a 8,7 mm. Contorno de 120x80
a 140x100 mm: la densidad bajaba de 53% a 36% y la caja sigue sin definir.

Sigue sin ruteo, sin vias y sin archivos de fabricacion. Falta ejecutar
Update PCB from Schematic en la GUI: KiCad no expone esa operacion por CLI.

Co-Authored-By: Claude Opus 5 <noreply@anthropic.com>
Parts:
- C9: value 10uF_PRELIMINAR -> 10uF_X5R_16V_1206; footprint rfid_eest3:CP_Radial_D5_P2.00_PLACEHOLDER_NO_FABRICAR -> Capacitor_SMD:C_1206_3216Metric

Commit message: Lleva J5 al borde y le pone conector con traba para el lector del marco
El RC522 va montado en el marco de la puerta y se conecta por cable. J5 estaba
en el medio de la placa, asi que el cable tenia que cruzar por encima de todo
el board. Se mueve al borde superior, junto a las borneras de sensores: todos
los cables que van hacia la puerta salen por el mismo lado y el borde inferior
queda para potencia y cerradura.

El footprint pasa de PinHeader_1x08_P2.54mm_Vertical a JST_XH_S8B-XH-A
horizontal: con traba y entrada lateral. Un header con jumpers dupont falla de
forma intermitente en algo que golpea cada vez que se abre la puerta.

La traza SPI sube de 8,7 a 43,7 mm. Es irrelevante: con el reloj a 1 MHz y las
resistencias serie de 33 ohm, el factor dominante son los 20-40 cm de cable, no
44 mm de pista.

Como el board conserva el footprint viejo hasta que se sincronice, la
colocacion reserva la union de ambas cajas. Sin eso J5 pisaba a J2 y el DRC
reportaba cortocircuito +3V3/GND de forma transitoria.

Se documentan en el informe las condiciones de instalacion del lector:
longitud de cable, separacion del metal del marco y desacoplo local.

Co-Authored-By: Claude Opus 5 <noreply@anthropic.com>
Parts:
- J5: value RC522_8PIN_3V3_PINOUT_PENDING -> RC522_8PIN_3V3_XH_CABLE_LECTOR; footprint Connector_PinHeader_2.54mm:PinHeader_1x08_P2.54mm_Vertical -> Connector_JST:JST_XH_S8B-XH-A_1x08_P2.50mm_Horizontal
