File: rfid-control-acceso-eest3/RESUMEN_ELECTRICO.kicad_sch (KiCad schematic)
At the start: 67 parts, among them J1 BOARD_12VDC_2.5A, J10 PIR_TAMPER, J11 PIR_PWR, J12 PIR_ALARM, J13 ESP32-S3-DevKitC-1_N16R8_44P, J2 BUCK?, J5 RC522_8PIN_3V3_XH_CABLE_LECTOR, J6 REED_NC, J8 CABINET_SENSOR, J9 LOCK_12V_1.8A_21.6W, Q1 AO3400A_PRELIM, Q2 AO3400A_PRELIM

Commit message: Unifica el resumen en un solo recuadro con titulo y epigrafe
La version anterior partia la hoja en seis cajas punteadas, una por bloque. Se
leia como seis esquemas puestos uno al lado del otro y no como el circuito que
son. Pasa a un unico recuadro con el titulo arriba y el nombre del esquema
abajo, que es el formato de lamina que se usa para entregar.

Los seis bloques siguen rotulados, pero ya sin caja propia: con 67 componentes
hace falta saber donde empieza cada parte, y el rotulo solo alcanza para eso
sin romper la unidad del dibujo.

El recuadro no esta escrito a mano: sale de los limites de lo que efectivamente
se dibujo, incluyendo el cuerpo de los simbolos y no solo sus pines, porque
mirando unicamente los pines el marco terminaba cortando los conectores del
borde. Si se mueve un bloque, el marco se reacomoda solo.

De paso, en el bloque de la cerradura Q2 quedaba conectado al nodo LOCK_OUT por
una diagonal corta. Ahora el drain cae exactamente sobre el riel y el nodo se
dibuja recto: el drain de Q2, el anodo de D4 y el pin 2 de J9 en una sola
linea, que es lo que conviene que se vea en ese punto del circuito.

TITULO y EPIGRAFE quedan como constantes arriba del script.

Las 34 redes siguen coincidiendo nodo por nodo con el esquema real.

Co-Authored-By: Claude Opus 5 <noreply@anthropic.com>
Other:
- note added: "CONTROL DE ACCESO RFID - E.E.S.T. N 3"
- note added: "D4 va pegado a J9: cuando Q2 corta, la corriente de la bobina"
- note added: "ESQUEMA ELECTRICO UNIFICADO - 67 componentes, 34 redes"
- note added: "encerrar la menor superficie posible."
- note added: "sigue circulando y se va por el diodo. Ese lazo tiene que"
- note removed: "D4 va pegado a J9: cuando Q2 corta, la corriente de la"
- note removed: "bobina sigue circulando y se va por el diodo. Ese lazo"
- note removed: "tiene que encerrar la menor superficie posible."
- moved on the sheet: BZ1, C11, D2, D3, D4, D9, J9, Q1, Q2, R3, R4, R5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

Commit message: Cablea el resumen de punta a punta y saca las etiquetas de señal
La version anterior tenia los bloques sueltos y unidos por etiquetas globales.
Era el mismo mecanismo que usa el esquema de origen, pero para una lamina de
una hoja no sirve: no se ve que va con que, hay que ir buscando el nombre
repetido en la otra punta.

Ahora hay cobre dibujado entre cada par de pines conectados. Cero etiquetas
globales, 232 cables. El ESP32 pasa al margen izquierdo, girado para que su
hilera impar mire hacia afuera, y de ahi sale un mazo de catorce canales
verticales que reparte cada señal a su bloque.

Lo unico que no va cableado son los rieles de alimentacion, que se resuelven
con simbolo, igual que en cualquier esquema de una hoja: una masa de treinta
nodos unida con cable no se lee. Los simbolos de +12V_LOCK, +12V_AUX, +12V_IN
y GND_POWER no existen en la biblioteca de KiCad y se derivan clonando la
forma del riel y renombrandola; el nombre de la red sale del nombre del pin, y
la biblioteca de sistema lo deja vacio, asi que sin ponerlo todos los rieles se
funden en una sola red.

Las catorce señales llevan etiqueta local encima del cable. No conectan nada
—el cobre ya esta— pero sin ellas KiCad bautiza la red Net-(J13-Pin_9) y deja
de significar algo.

Se agrega tools/verificar_cortos.py. Al cablear todo aparecio un problema que
con etiquetas no existia: dos redes que se tocan por geometria. Encontro ocho
cortocircuitos, todos de la misma familia —un tramo vertical de 8 mm que sale
de un pin y entra en la fila del vecino, con paso de 2,54 mm— y ademas dos
errores propios: R14 y R16 conectadas al reves, y el riel de masa de potencia
pasando a traves de NT1 en vez de morir en su pin 1, que lo cortocircuitaba.
Ninguno de los tres se veia en el dibujo.

Los tramos de alimentacion sobre hileras de pines pasan a medir 1,27 mm, menos
que el paso: asi no hay forma de que uno suba y otro baje y se toquen.

Las 34 redes siguen coincidiendo nodo por nodo con el esquema real.

Co-Authored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
Other:
- note added: "D4 pegado a J9: el lazo de recirculacion tiene que ser chico."
- note added: "ESQUEMA ELECTRICO INTEGRADO - 67 componentes, 34 redes, todo cableado"
- note added: "Se alimenta con +5V por el pin 41. R17 sostiene EN."
- note added: "alimentacion del PIR"
- note removed: "C5 desacopla, R17 mantiene EN arriba."
- note removed: "D4 va pegado a J9: cuando Q2 corta, la corriente de la bobina"
- note removed: "D9 absorbe el pico del buzzer al cortar."
- note removed: "ESQUEMA ELECTRICO UNIFICADO - 67 componentes, 34 redes"
- note removed: "Se alimenta con +5V por el pin 41."
- note removed: "alimentacion del PIR (12 V por F2)"
- note removed: "encerrar la menor superficie posible."
- note removed: "sigue circulando y se va por el diodo. Ese lazo tiene que"
- moved on the sheet: BZ1, C1, C10, C11, C2, C3, C4, C5, C6, C7, C8, C9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
